Commit message: fixed package names as robolaunch_cloudy

File: robolaunch_cloudy_description/sensors/generic_laser.urdf.xacro (robot description, xacro)
@@ -1,5 +1,5 @@
 <?xml version="1.0"?>
 <robot xmlns:xacro="http://ros.org/wiki/xacro">
-  <xacro:include filename="$(find robolaunch_diffbot_description)/sensors/laser.urdf.xacro" />
+  <xacro:include filename="$(find robolaunch_cloudy_description)/sensors/laser.urdf.xacro" />
   <xacro:macro name="generic_laser" params="*origin">
     <xacro:laser

File: robolaunch_cloudy_description/sensors/laser.urdf.xacro (robot description, xacro)
@@ -6,5 +6,5 @@
         <origin xyz="-0.05 0.03 -0.02" rpy="1.57 0 0"/>
         <geometry>
-                <mesh scale="${scale_ratio} ${scale_ratio} ${scale_ratio}" filename="file://$(find robolaunch_diffbot_description)/urdf/meshes/lidar.stl" />
+                <mesh scale="${scale_ratio} ${scale_ratio} ${scale_ratio}" filename="file://$(find robolaunch_cloudy_description)/urdf/meshes/lidar.stl" />
         </geometry>
         <material name="green">

File: robolaunch_cloudy_description/urdf/diffbot_system.urdf.xacro (robot description, xacro)
@@ -3,5 +3,5 @@
 <!--
 Copied and modified from ROS1 example -
-https://github.com/ros-simulation/gazebo_ros_demos/blob/kinetic-devel/robolaunch_diffbot_description/urdf/diffbot.xacro
+https://github.com/ros-simulation/gazebo_ros_demos/blob/kinetic-devel/robolaunch_cloudy_description/urdf/diffbot.xacro
 -->
 <robot xmlns:xacro="http://www.ros.org/wiki/xacro" name="diffdrive_robot">
@@ -11,16 +11,16 @@
   <xacro:arg name="fake_sensor_commands" default="false" />
   <xacro:arg name="prefix" default="" />
-  <xacro:include filename="$(find robolaunch_diffbot_description)/urdf/robot_core.xacro" />
+  <xacro:include filename="$(find robolaunch_cloudy_description)/urdf/robot_core.xacro" />
 <xacro:generic_laser>
         <xacro:insert_block name="laser_pose" />
     </xacro:generic_laser>
   <!-- Import all Gazebo-customization elements, including Gazebo colors -->
-<!--   <xacro:include filename="$(find robolaunch_diffbot_description)/gazebo/diffbot.gazebo.xacro" />
+<!--   <xacro:include filename="$(find robolaunch_cloudy_description)/gazebo/diffbot.gazebo.xacro" />
  -->
   <!-- Import Rviz colors -->
-<!--   <xacro:include filename="$(find robolaunch_diffbot_description)/gazebo/diffbot.materials.xacro" />
+<!--   <xacro:include filename="$(find robolaunch_cloudy_description)/gazebo/diffbot.materials.xacro" />
  -->
   <!-- Import diffbot ros2_control description -->
-  <xacro:include filename="$(find robolaunch_diffbot_description)/ros2_control/diffbot_system.ros2_control.xacro" />
+  <xacro:include filename="$(find robolaunch_cloudy_description)/ros2_control/diffbot_system.ros2_control.xacro" />
 <!--   <xacro:diffbot prefix="$(arg prefix)" />
  -->

File: robolaunch_cloudy_description/urdf/robot_core.xacro (robot description, xacro)
@@ -2,6 +2,6 @@
 <robot xmlns:xacro="http://www.ros.org/wiki/xacro" >
     <xacro:include filename="inertial_macros.xacro"/>
-    <xacro:include filename="$(find robolaunch_diffbot_description)/sensors/generic_laser.urdf.xacro" />
-    <xacro:include filename="$(find robolaunch_diffbot_description)/urdf/properties.urdf.xacro" />
+    <xacro:include filename="$(find robolaunch_cloudy_description)/sensors/generic_laser.urdf.xacro" />
+    <xacro:include filename="$(find robolaunch_cloudy_description)/urdf/properties.urdf.xacro" />
    <xacro:property name="scale_ratio" value="0.0015" />
    <link name="base_footprint"/>
@@ -39,5 +39,5 @@
             <origin xyz="0 0.15 0" rpy="1.57 0 0"/>
             <geometry>
-                <mesh scale="${scale_ratio} ${scale_ratio} ${scale_ratio}" filename="file://$(find robolaunch_diffbot_description)/urdf/meshes/body.stl"/>
+                <mesh scale="${scale_ratio} ${scale_ratio} ${scale_ratio}" filename="file://$(find robolaunch_cloudy_description)/urdf/meshes/body.stl"/>
             </geometry>
             <material name="gray"/>
@@ -68,5 +68,5 @@
         <visual>
             <geometry>
-                <mesh scale="${scale_ratio} ${scale_ratio} ${scale_ratio}" filename="file://$(find robolaunch_diffbot_description)/urdf/meshes/wheel.stl" />
+                <mesh scale="${scale_ratio} ${scale_ratio} ${scale_ratio}" filename="file://$(find robolaunch_cloudy_description)/urdf/meshes/wheel.stl" />
             </geometry>
             <material name="white"/>
@@ -95,5 +95,5 @@
         <visual>
             <geometry>
-                <mesh scale="${scale_ratio} ${scale_ratio} ${scale_ratio}" filename="file://$(find robolaunch_diffbot_description)/urdf/meshes/wheel.stl" />
+                <mesh scale="${scale_ratio} ${scale_ratio} ${scale_ratio}" filename="file://$(find robolaunch_cloudy_description)/urdf/meshes/wheel.stl" />
             </geometry>
             <origin xyz="-0.049 -0.049 0" rpy="0 ${pi/2} 0" />
