Commit message: added intel realsense d435i camera on simulation

File: robolaunch_cloudy_description/sensors/depth_sensor.urdf.xacro (robot description, xacro)
@@ -4,8 +4,8 @@
     <link name="camera_link">
       <visual>
-        <origin xyz="0 0 0" rpy="0 0 0"/>
+        <origin xyz="-0.05 -0.105 0" rpy="1.57 0 1.57"/>
         <geometry>
-          <box size="0.030 0.124 0.030"/>
-          <!-- <mesh filename="" scale="0.001 0.001 0.001"/> -->
+<!--      <box size="0.030 0.124 0.030"/> -->
+          <mesh scale="${scale_ratio} ${scale_ratio} ${scale_ratio}" filename="file://$(find robolaunch_cloudy_description)/urdf/meshes/realsense.stl" />
         </geometry>
         <material name="red">

File: robolaunch_cloudy_description/urdf/diffbot_system.urdf.xacro (robot description, xacro)
@@ -15,4 +15,7 @@
         <xacro:insert_block name="laser_pose" />
     </xacro:generic_laser>
+    <xacro:depth_sensor>
+        <xacro:insert_block name="depth_sensor_pose" />
+    </xacro:depth_sensor>
   <!-- Import all Gazebo-customization elements, including Gazebo colors -->
 <!--   <xacro:include filename="$(find robolaunch_cloudy_description)/gazebo/diffbot.gazebo.xacro" />

File: robolaunch_cloudy_description/urdf/robot.urdf.xacro (robot description, xacro)
@@ -4,12 +4,9 @@
     <xacro:include filename="robot_core.xacro"/>
     <xacro:include filename="gazebo_control.xacro"/>
-  <xacro:property name="depth_sensor_pose">
-    <origin xyz="-0.065 0 0.255" rpy="0 0 0"/>
-  </xacro:property>
     <xacro:generic_laser>
         <xacro:insert_block name="laser_pose" />
     </xacro:generic_laser>
-  <xacro:depth_sensor>
-    <xacro:insert_block name="depth_sensor_pose" />
-  </xacro:depth_sensor>
+    <xacro:depth_sensor>
+        <xacro:insert_block name="depth_sensor_pose" />
+    </xacro:depth_sensor>
 </robot>

File: robolaunch_cloudy_description/urdf/robot_core.xacro (robot description, xacro)
@@ -5,4 +5,7 @@
     <xacro:include filename="$(find robolaunch_cloudy_description)/urdf/properties.urdf.xacro" />
     <xacro:include filename="$(find robolaunch_cloudy_description)/sensors/depth_sensor.urdf.xacro" />
+    <xacro:property name="depth_sensor_pose">
+        <origin xyz="0.4 0 0.05" rpy="0 0 0"/>
+    </xacro:property>
    <xacro:property name="scale_ratio" value="0.0015" />
    <link name="base_footprint"/>

Commit message: change lidar and depth camera color and replacement the lidar

File: robolaunch_cloudy_description/sensors/depth_sensor.urdf.xacro (robot description, xacro)
@@ -9,7 +9,7 @@
           <mesh scale="${scale_ratio} ${scale_ratio} ${scale_ratio}" filename="file://$(find robolaunch_cloudy_description)/urdf/meshes/realsense.stl" />
         </geometry>
-        <material name="red">
-          <color rgba="0.416 0.051 0.047 1.0"/>
-        </material>
+  <material name="lightgray">
+        <color rgba="0.6 0.6 0.6 1"/>
+    </material>
       </visual>
       <collision>
@@ -27,14 +27,4 @@
       </inertial>
     </link>
-    <gazebo reference="camera_link">
-      <visual>
-        <material>
-          <ambient>0.416 0.051 0.047 1.0</ambient>
-          <diffuse>0.416 0.051 0.047 1.0</diffuse>
-          <specular>0.416 0.051 0.047 1.0</specular>
-          <emissive>0.416 0.051 0.047 1.0</emissive>
-        </material>
-      </visual>
-    </gazebo>rgb(213,28,40)
     <joint name="camera_to_base_link" type="fixed">
       <parent link="base_link"/>

File: robolaunch_cloudy_description/sensors/laser.urdf.xacro (robot description, xacro)
@@ -4,14 +4,15 @@
     <link name="${frame_id}">
       <visual>
-        <origin xyz="-0.05 0.03 -0.02" rpy="1.57 0 0"/>
+        <origin xyz="0.04 -0.038 -0.08" rpy="1.57 0 3.14"/>
         <geometry>
-                <mesh scale="${scale_ratio} ${scale_ratio} ${scale_ratio}" filename="file://$(find robolaunch_cloudy_description)/urdf/meshes/lidar.stl" />
-        </geometry>
-        <material name="green">
-            <color rgba="0.003 0.639 0.223 1.0"/>
-        </material>
+              <mesh scale="${scale_ratio} ${scale_ratio} ${scale_ratio}" filename="file://$(find robolaunch_cloudy_description)/urdf/meshes/lidar.stl" />
+           <!--   <cylinder radius="0.0375" length="0.05"/> -->
+         </geometry>
+  <material name="darkgray">
+        <color rgba="0.2 0.2 0.2 1"/>
+    </material>
       </visual>
       <collision>
-        <origin xyz="0 0 -0.025" rpy="0 0 0"/>
+        <origin xyz="0 0 0" rpy="0 0 0"/>
         <geometry>
           <cylinder radius="0.0375" length="0.05"/>
@@ -27,14 +28,8 @@
     </link>
     <gazebo reference="${frame_id}">
-      <visual>
-        <material>
-          <ambient>0.003 0.639 0.223 1.0</ambient>
-          <diffuse>0.003 0.639 0.223 1.0</diffuse>
-          <specular>0.003 0.639 0.223 1.0</specular>
-          <emissive>0.0 0.0 0.0 0.0</emissive>
-        </material>
-      </visual>
+    <material>Gazebo/Black</material>
     </gazebo>
     <joint name="${frame_id}_to_base_link" type="fixed">
+      <origin xyz="0 -0.01 0.26" rpy="0 0 0"/>
       <parent link="base_link"/>
       <child link="${frame_id}"/>
@@ -46,5 +41,5 @@
         <update_rate>${update_rate}</update_rate>
         <pose>0 0 0 0 0 0</pose>
-        <visualize>false</visualize>
+        <visualize>false</visualize> <!-- if you want to see laser scan lines into the gazebo you should enable this -->
         <ray>
           <scan>

File: robolaunch_cloudy_description/urdf/properties.urdf.xacro (robot description, xacro)
@@ -2,5 +2,5 @@
 <robot xmlns:xacro="http://ros.org/wiki/xacro">
   <xacro:property name="laser_pose">
-    <origin xyz="-0.01 -0.018 0.2" rpy="0 0 3.14"/>
+    <origin xyz="0 0 0" rpy="0 0 0"/>
   </xacro:property>
 </robot>
