Commit message: cloudy v2 urdf update and laser filter package

File: robolaunch_cloudy_description/sensors/laser.urdf.xacro (robot description, xacro)
@@ -4,5 +4,5 @@
     <link name="${frame_id}">
       <visual>
-        <origin xyz="0.04 -0.038 -0.08" rpy="1.57 0 3.14"/>
+        <origin xyz="0.04 -0.038 -0.03" rpy="1.57 0 3.14"/>
         <geometry>
               <mesh scale="${scale_ratio} ${scale_ratio} ${scale_ratio}" filename="file://$(find robolaunch_cloudy_description)/urdf/meshes/lidar.stl" />
@@ -14,7 +14,7 @@
       </visual>
       <collision>
-        <origin xyz="0 0 0" rpy="0 0 0"/>
+        <origin xyz="0.02 0 -0.018" rpy="0 0 0"/>
         <geometry>
-          <cylinder radius="0.0375" length="0.05"/>
+          <cylinder radius="0.0375" length="0.02"/>
         </geometry>
       </collision>
@@ -31,5 +31,5 @@
     </gazebo>
     <joint name="${frame_id}_to_base_link" type="fixed">
-      <origin xyz="0 -0.01 0.26" rpy="0 0 0"/>
+      <origin xyz="0.32 -0.01 0.085" rpy="0 0 0"/>
       <parent link="base_link"/>
       <child link="${frame_id}"/>

File: robolaunch_cloudy_description/urdf/gazebo_control.xacro (robot description, xacro)
@@ -5,6 +5,6 @@
         <left_joint>left_wheel_joint</left_joint>
         <right_joint>right_wheel_joint</right_joint>
-        <wheel_separation>0.25</wheel_separation>
-        <wheel_diameter>0.07</wheel_diameter>
+        <wheel_separation>0.255</wheel_separation>
+        <wheel_diameter>0.066</wheel_diameter>
         <!--limits-->
         <max_wheel_torque>200</max_wheel_torque>

File: robolaunch_cloudy_description/urdf/robot_core.xacro (robot description, xacro)
@@ -6,5 +6,5 @@
     <xacro:include filename="$(find robolaunch_cloudy_description)/sensors/depth_sensor.urdf.xacro" />
     <xacro:property name="depth_sensor_pose">
-        <origin xyz="0.4 0 0.05" rpy="0 0 0"/>
+        <origin xyz="0.38 0 0.11" rpy="0 -0.15 0"/>
     </xacro:property>
    <xacro:property name="scale_ratio" value="0.0015" />
@@ -37,22 +37,22 @@
         <parent link="base_link"/>
         <child link="chassis"/>
-        <origin xyz="-0.1 0 0"/>
+        <origin xyz="0 -0.2 0" rpy="0 0 1.57 "/>
     </joint>
     <link name="chassis">
         <visual>
-            <origin xyz="0 0.15 0" rpy="1.57 0 0"/>
+            <origin xyz="0 0.15 -0.02" rpy="1.57 0 0"/>
             <geometry>
-                <mesh scale="${scale_ratio} ${scale_ratio} ${scale_ratio}" filename="file://$(find robolaunch_cloudy_description)/urdf/meshes/body.stl"/>
+                <mesh scale="${scale_ratio} ${scale_ratio} ${scale_ratio}" filename="file://$(find robolaunch_cloudy_description)/urdf/meshes/body_v2.stl"/>
             </geometry>
             <material name="gray"/>
         </visual>
         <collision>
-            <origin xyz="0.25 0 0.075"/>
+            <origin xyz="0.20 -0.1 0.075"/>
             <geometry>
-                <box size="0.5 0.3 0.15"/>
+                <box size="0.3 0.5 0.15"/>
             </geometry>
         </collision>
         <xacro:inertial_box mass="0.5" x="0.3" y="0.3" z="0.15">
-            <origin xyz="0.15 0 0.075" rpy="0 0 0"/>
+            <origin xyz="0.15 0 0.072" rpy="0 0 0"/>
         </xacro:inertial_box>
     </link>
@@ -66,5 +66,5 @@
         <parent link="base_link"/>
         <child link="left_wheel"/>
-        <origin xyz="0.145 0.14 0.048" rpy="-${pi/2} 0 0" />
+        <origin xyz="0.11 0.14 0.046" rpy="-${pi/2} 0 0" />
         <axis xyz="0 0 1"/>
     </joint>
@@ -72,8 +72,8 @@
         <visual>
             <geometry>
-                <mesh scale="${scale_ratio} ${scale_ratio} ${scale_ratio}" filename="file://$(find robolaunch_cloudy_description)/urdf/meshes/wheel.stl" />
+                <mesh scale="${scale_ratio} ${scale_ratio} ${scale_ratio}" filename="file://$(find robolaunch_cloudy_description)/urdf/meshes/wheel_v2.stl" />
             </geometry>
             <material name="white"/>
-            <origin xyz="-0.049 -0.049 0" rpy="0 ${pi/2} 0" />
+            <origin xyz="-0.067 -0.05 -0.15" rpy="0 0 0" />
         </visual>
         <collision>
@@ -93,5 +93,5 @@
         <parent link="base_link"/>
         <child link="right_wheel"/>
-        <origin xyz="0.145 -0.14 0.048" rpy="-${pi/2} 0 0" />
+        <origin xyz="0.11 -0.14 0.046" rpy="-${pi/2} 0 0" />
         <axis xyz="0 0 1"/>
     </joint>
@@ -99,7 +99,7 @@
         <visual>
             <geometry>
-                <mesh scale="${scale_ratio} ${scale_ratio} ${scale_ratio}" filename="file://$(find robolaunch_cloudy_description)/urdf/meshes/wheel.stl" />
+                <mesh scale="${scale_ratio} ${scale_ratio} ${scale_ratio}" filename="file://$(find robolaunch_cloudy_description)/urdf/meshes/wheel_v2.stl" />
             </geometry>
-            <origin xyz="-0.049 -0.049 0" rpy="0 ${pi/2} 0" />
+            <origin xyz="-0.067 -0.05 -0.15" rpy="0 0 0" />
             <material name="white"/>
         </visual>

Commit message: minor bug fix

File: robolaunch_cloudy_description/sensors/laser.urdf.xacro (robot description, xacro)
@@ -31,5 +31,5 @@
     </gazebo>
     <joint name="${frame_id}_to_base_link" type="fixed">
-      <origin xyz="0.32 -0.01 0.085" rpy="0 0 0"/>
+      <origin xyz="0.32 -0.01 0.085" rpy="0 0 3.14159"/>
       <parent link="base_link"/>
       <child link="${frame_id}"/>

Commit message: physical arcelik support

File: robolaunch_cloudy_description/sensors/laser.urdf.xacro (robot description, xacro)
@@ -31,5 +31,5 @@
     </gazebo>
     <joint name="${frame_id}_to_base_link" type="fixed">
-      <origin xyz="0.32 -0.01 0.085" rpy="0 0 3.14159"/>
+      <origin xyz="0.25 -0.01 0.35" rpy="0 0 3.14159"/>
       <parent link="base_link"/>
       <child link="${frame_id}"/>

Commit message: refactor(parameters): update laser filter params

File: robolaunch_cloudy_description/sensors/laser.urdf.xacro (robot description, xacro)
@@ -31,5 +31,5 @@
     </gazebo>
     <joint name="${frame_id}_to_base_link" type="fixed">
-      <origin xyz="0.25 -0.01 0.35" rpy="0 0 3.14159"/>
+      <origin xyz="0.25 -0.01 0.35" rpy="0 0 0"/>
       <parent link="base_link"/>
       <child link="${frame_id}"/>

Commit message: unstable features that are not ready to merge to main yet

File: robolaunch_cloudy_description/sensors/laser.urdf.xacro (robot description, xacro)
@@ -31,5 +31,5 @@
     </gazebo>
     <joint name="${frame_id}_to_base_link" type="fixed">
-      <origin xyz="0.25 -0.01 0.35" rpy="0 0 3.14159"/>
+      <origin xyz="0.32 -0.01 0.2" rpy="0 0 3.14159"/>
       <parent link="base_link"/>
       <child link="${frame_id}"/>

File: robolaunch_cloudy_description/urdf/robots/arcelik/base.urdf.xacro (robot description, xacro)
@@ -29,26 +29,4 @@
                  izz="${(1/12) * mass * ((length * length) + (width  * width))}"/>
       </inertial>
-    </link>
-    <link name="rplidar">
-      <inertial>
-        <origin xyz="0 0 0" rpy="0 0 0"/>
-        <mass value="1"/>
-        <inertia ixx="0.1"  ixy="0"  ixz="0" iyy="0.1" iyz="0" izz="0.1" />
-      </inertial>
-      <visual>
-        <origin xyz="0 0 ${yukseklik}" rpy="0 0 0" />
-        <geometry>
-		<mesh scale="${scale_ratio} ${scale_ratio} ${scale_ratio}" filename="$(find robolaunch_cloudy_description)/urdf/meshes/arcelik/lidar.stl"/>
-        </geometry>
-        <material name="yellow">
-          <color rgba="0.1 0.6627 0.6627 1.0"/>
-        </material>
-      </visual>
-      <collision>
-        <origin xyz="0 0 ${yukseklik}" rpy="0 0 0"/>
-        <geometry>
-          <box size="0.1 0.1 0.1" />
-        </geometry>
-      </collision>
     </link>
         <link name="iskelet">
@@ -111,9 +89,4 @@
       <origin xyz="0 0 ${wheel_radius - wheel_pos_z}" rpy="0 0 0"/>
     </joint>
-        <joint name="lidar_joint" type="fixed">
-      <parent link="base_link"/>
-      <child link="rplidar"/>
-      <origin xyz="0.05 0.015 0.29" rpy="0 0 1.57"/>
-    </joint>
         <joint name="rig_joint" type="fixed">
       <parent link="base_link"/>
