Commit message: add depth camera and fix package name as robolaunch_cloudy

File: robolaunch_cloudy_description/urdf/robot.urdf.xacro (robot description, xacro)
@@ -4,6 +4,12 @@
     <xacro:include filename="robot_core.xacro"/>
     <xacro:include filename="gazebo_control.xacro"/>
+  <xacro:property name="depth_sensor_pose">
+    <origin xyz="-0.065 0 0.255" rpy="0 0 0"/>
+  </xacro:property>
     <xacro:generic_laser>
         <xacro:insert_block name="laser_pose" />
     </xacro:generic_laser>
+  <xacro:depth_sensor>
+    <xacro:insert_block name="depth_sensor_pose" />
+  </xacro:depth_sensor>
 </robot>

File: robolaunch_cloudy_description/urdf/robot_core.xacro (robot description, xacro)
@@ -4,4 +4,5 @@
     <xacro:include filename="$(find robolaunch_cloudy_description)/sensors/generic_laser.urdf.xacro" />
     <xacro:include filename="$(find robolaunch_cloudy_description)/urdf/properties.urdf.xacro" />
+    <xacro:include filename="$(find robolaunch_cloudy_description)/sensors/depth_sensor.urdf.xacro" />
    <xacro:property name="scale_ratio" value="0.0015" />
    <link name="base_footprint"/>
