Commit message: barcode world and fix robot lidar positions

File: robolaunch_cloudy_description/urdf/robots/arcelik/base.urdf.xacro (robot description, xacro)
@@ -9,5 +9,5 @@
         <origin xyz="-0.3 0 ${yukseklik}" rpy="0 0 1.57"/>
         <geometry>
-		<mesh scale="${scale_ratio} ${scale_ratio} ${scale_ratio}" filename="$(find robolaunch_cloudy_description)/urdf/meshes/arcelik/chassis_red.stl"/>
+		<mesh scale="${scale_ratio} ${scale_ratio} ${scale_ratio}" filename="file://$(find robolaunch_cloudy_description)/urdf/meshes/arcelik/chassis_red.stl"/>
           <!-- <mesh ="" scale="0.001 0.001 0.001"/> -->
         </geometry>
@@ -39,5 +39,5 @@
         <origin xyz="0 0 ${yukseklik}" rpy="0 0 0" />
         <geometry>
-          <mesh scale="${scale_ratio} ${scale_ratio} ${scale_ratio}" filename="$(find robolaunch_cloudy_description)/urdf/meshes/arcelik/son_rigs.stl"/>
+          <mesh scale="${scale_ratio} ${scale_ratio} ${scale_ratio}" filename="file://$(find robolaunch_cloudy_description)/urdf/meshes/arcelik/son_rigs.stl"/>
         </geometry>
         <material name="yellow">
@@ -61,5 +61,5 @@
         <origin xyz="0 0 ${yukseklik}" rpy="0 0 0" />
         <geometry>
-		<mesh scale="${scale_ratio} ${scale_ratio} ${scale_ratio}" filename="$(find robolaunch_cloudy_description)/urdf/meshes/arcelik/UstPlaka2.stl"/>
+		<mesh scale="${scale_ratio} ${scale_ratio} ${scale_ratio}" filename="file://$(find robolaunch_cloudy_description)/urdf/meshes/arcelik/UstPlaka2.stl"/>
         </geometry>
         <material name="yellow">

File: robolaunch_cloudy_description/urdf/robots/arcelik/mecanum.urdf.xacro (robot description, xacro)
@@ -6,6 +6,6 @@
   <xacro:include filename="$(find robolaunch_cloudy_description)/urdf/robots/arcelik/mecanum_wheel2.urdf.xacro" />
   <xacro:include filename="$(find robolaunch_cloudy_description)/sensors/imu.urdf.xacro" />
-  <xacro:include filename="$(find robolaunch_cloudy_description)/sensors/generic_laser.urdf.xacro" />
-  <xacro:include filename="$(find robolaunch_cloudy_description)/sensors/depth_sensor.urdf.xacro" />
+  <xacro:include filename="$(find robolaunch_cloudy_description)/sensors/laser_arcelik.xacro" />
+  <xacro:include filename="$(find robolaunch_cloudy_description)/sensors/depth_sensor_arcelik.xacro" />
   <xacro:include filename="$(find robolaunch_cloudy_description)/urdf/robots/arcelik/suspention.urdf.xacro" />
   <xacro:include filename="$(find robolaunch_cloudy_description)/urdf/omni_drive.urdf.xacro" />

File: robolaunch_cloudy_description/urdf/robots/arcelik/mecanum_properties.urdf.xacro (robot description, xacro)
@@ -5,5 +5,5 @@
   <xacro:property name="base_height" value="0.259" />
   <xacro:property name="base_mass" value="10" />
-  <xacro:property name="wheel_radius" value="0.16162" />
+  <xacro:property name="wheel_radius" value="0.14162" />
   <xacro:property name="wheel_width" value="0.07" />
   <xacro:property name="wheel_pos_x" value="0.530" />

File: robolaunch_cloudy_description/urdf/robots/arcelik/mecanum_wheel.urdf.xacro (robot description, xacro)
@@ -7,5 +7,5 @@
         <origin xyz="0 0.1 0" rpy="${yon} 0 0"/>
         <geometry>
-		<mesh scale="${scale_ratio} ${scale_ratio} ${scale_ratio}" filename="$(find robolaunch_cloudy_description)/urdf/meshes/arcelik/teker_cw.dae"/>
+		<mesh scale="${scale_ratio} ${scale_ratio} ${scale_ratio}" filename="file://$(find robolaunch_cloudy_description)/urdf/meshes/arcelik/teker_cw.dae"/>
         </geometry>
         <material name="blue">
@@ -14,5 +14,5 @@
       </visual>
       <collision>
-        <origin xyz="0 0 0" rpy="${yon} 0 0"/>
+        <origin xyz="0 0.1 0" rpy="${yon} 0 0"/>
         <geometry>
           <cylinder radius="${radius}" length="${width}"/>
@@ -28,6 +28,6 @@
     </link>
     <gazebo reference="${side}_wheel_link">
-        <mu1>0.2</mu1>
-        <mu2>0.2</mu2>
+        <mu1>0.5</mu1>
+        <mu2>0.5</mu2>
     </gazebo>
     <gazebo reference="${side}_wheel_link">

File: robolaunch_cloudy_description/urdf/robots/arcelik/mecanum_wheel2.urdf.xacro (robot description, xacro)
@@ -7,5 +7,5 @@
         <origin xyz="0 0.21 0" rpy="${yon} 0 0"/>
         <geometry>
-		<mesh scale="${scale_ratio} ${scale_ratio} ${scale_ratio}" filename="$(find robolaunch_cloudy_description)/urdf/meshes/arcelik/teker_cw.dae"/>
+		<mesh scale="${scale_ratio} ${scale_ratio} ${scale_ratio}" filename="file://$(find robolaunch_cloudy_description)/urdf/meshes/arcelik/teker_cw.dae"/>
         </geometry>
         <material name="blue">
@@ -14,5 +14,5 @@
       </visual>
       <collision>
-        <origin xyz="0 0 0" rpy="${yon} 0 0"/>
+        <origin xyz="0 0.2 0" rpy="${yon} 0 0"/>
         <geometry>
           <cylinder radius="${radius}" length="${width}"/>
@@ -28,6 +28,6 @@
     </link>
     <gazebo reference="${side}_wheel_link">
-        <mu1>0.2</mu1>
-        <mu2>0.2</mu2>
+        <mu1>0.5</mu1>
+        <mu2>0.5</mu2>
     </gazebo>
     <gazebo reference="${side}_wheel_link">

File: robolaunch_cloudy_description/urdf/robots/arcelik/suspention.urdf.xacro (robot description, xacro)
@@ -6,5 +6,5 @@
         <origin xyz="0 0 0" rpy="${yon} ${yonp} 0"/>
         <geometry>
-		<mesh scale="0.0015 0.0015 0.0015" filename="package://linorobot2_description/urdf/mech/mesh/suspention_son.dae"/>
+		<mesh scale="0.0015 0.0015 0.0015" filename="file://$(find robolaunch_cloudy_description)/urdf/meshes/arcelik/suspention_son.dae"/>
         </geometry>
         <material name="blue">
@@ -15,5 +15,5 @@
         <origin xyz="0 0 0" rpy="${yon} 0 0"/>
         <geometry>
-          <cylinder radius="${radius}" length="${width}"/>
+          <cylinder radius="0.02" length="0.02"/>
         </geometry>
       </collision>

File: robolaunch_cloudy_description/urdf/robots/cloudy_v1_core.xacro (robot description, xacro)
@@ -2,7 +2,7 @@
 <robot xmlns:xacro="http://www.ros.org/wiki/xacro" >
     <xacro:include filename="$(find robolaunch_cloudy_description)/urdf/inertial_macros.xacro"/>
-    <xacro:include filename="$(find robolaunch_cloudy_description)/sensors/generic_laser.urdf.xacro" />
+    <xacro:include filename="$(find robolaunch_cloudy_description)/sensors/generic_laser_cloudy_v1.xacro" />
     <xacro:include filename="$(find robolaunch_cloudy_description)/urdf/robots/cloudy_v1_properties.urdf.xacro" />
-    <xacro:include filename="$(find robolaunch_cloudy_description)/sensors/depth_sensor.urdf.xacro" />
+    <xacro:include filename="$(find robolaunch_cloudy_description)/sensors/depth_sensor_cloudy_v1.xacro" />
     <xacro:property name="depth_sensor_pose">
         <origin xyz="0.4 0 0.05" rpy="0 0 0"/>

File: robolaunch_cloudy_description/urdf/robots/cloudy_v2_core.xacro (robot description, xacro)
@@ -2,7 +2,7 @@
 <robot xmlns:xacro="http://www.ros.org/wiki/xacro" >
     <xacro:include filename="$(find robolaunch_cloudy_description)/urdf/inertial_macros.xacro"/>
-    <xacro:include filename="$(find robolaunch_cloudy_description)/sensors/generic_laser.urdf.xacro" />
+    <xacro:include filename="$(find robolaunch_cloudy_description)/sensors/generic_laser_cloudy_v2.xacro" />
     <xacro:include filename="$(find robolaunch_cloudy_description)/urdf/robots/cloudy_v2_properties.urdf.xacro" />
-    <xacro:include filename="$(find robolaunch_cloudy_description)/sensors/depth_sensor.urdf.xacro" />
+    <xacro:include filename="$(find robolaunch_cloudy_description)/sensors/depth_sensor_cloudy_v2.xacro" />
     <xacro:property name="depth_sensor_pose">
         <origin xyz="0.38 0 0.11" rpy="0 -0.15 0"/>
