Commit message: fixed cloudy_v2 lidar position

File: robolaunch_cloudy_description/urdf/robots/cloudy_v2_core.xacro (robot description, xacro)
@@ -66,5 +66,5 @@
         <parent link="base_link"/>
         <child link="left_wheel"/>
-        <origin xyz="0.11 0.14 0.046" rpy="-${pi/2} 0 0" />
+        <origin xyz="0.11 0.14 0.048" rpy="-${pi/2} 0 0" />
         <axis xyz="0 0 1"/>
     </joint>
@@ -93,5 +93,5 @@
         <parent link="base_link"/>
         <child link="right_wheel"/>
-        <origin xyz="0.11 -0.14 0.046" rpy="-${pi/2} 0 0" />
+        <origin xyz="0.11 -0.14 0.048" rpy="-${pi/2} 0 0" />
         <axis xyz="0 0 1"/>
     </joint>

Commit message: first

File: robolaunch_cloudy_description/urdf/robots/cloudy_v2_core.xacro (robot description, xacro)
@@ -31,5 +31,5 @@
       <parent link="base_footprint"/>
       <child link="base_link"/>
-      <origin xyz="0 0 0.035" rpy="0 0 0"/>
+      <origin xyz="0 0 0.2" rpy="0 0 0"/>
     </joint>
     <!-- CHASSIS LINK -->
